Commit message: [iris] Reposition Hokuyo.

File: robots_description/models/iris_hokuyo/model.xacro (robot description, xacro)
@@ -52,5 +52,5 @@
   <joint name="hokuyo_joint" type="fixed">
     <axis xyz="0 1 0" />
-    <origin xyz="0 0 .1" rpy="0 -0.872665 3.14"/>
+    <origin xyz="0.1 0 .1" rpy="0 -0.872665 0"/>
     <parent link="base_link"/>
     <child link="hokuyo"/>
